File: dev/hardware/Power.kicad_sch (KiCad schematic)
At the start: 6 parts, among them J301 DC IN, U301 LF33_TO220

Commit message: Finalized physical layout
Parts:
- added Q301: IPP80P03P4L-04, Package_TO_SOT_THT:TO-220-3_Horizontal_TabDown, symbol jcap-symbols:IPP80P03P4L-04
Connections:
- net GND: now also Q301.1 (G)
- net at C?.2, J301.1: now also Q301.3 (S); no longer U301.1 (IN)
- new net: Q301.2 (D), U301.1 (IN)
Other:
- moved on the sheet: C?, J301
Changed lines of the file:
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@@
 (kicad_sch (version 20230121) (generator eeschema)
   (paper "A4")
-  (junction (at 124.46 92.71) (diameter 0) (color 0 0 0 0)
+  (junction (at 102.87 92.71) (diameter 0) (color 0 0 0 0)
+  )
+  (junction (at 120.65 102.87) (diameter 0) (color 0 0 0 0)
   )
   (junction (at 180.34 87.63) (diameter 0) (color 0 0 0 0)
@@
   (junction (at 180.34 102.87) (diameter 0) (color 0 0 0 0)
   )
-  (junction (at 130.81 102.87) (diameter 0) (color 0 0 0 0)
-  )
-  (junction (at 130.81 87.63) (diameter 0) (color 0 0 0 0)
+  (junction (at 109.22 102.87) (diameter 0) (color 0 0 0 0)
+  )
+  (junction (at 109.22 87.63) (diameter 0) (color 0 0 0 0)
   )
   (junction (at 173.99 102.87) (diameter 0) (color 0 0 0 0)
@@
   (junction (at 191.77 87.63) (diameter 0) (color 0 0 0 0)
   )
+  (junction (at 134.62 87.63) (diameter 0) (color 0 0 0 0)
+  )
   (wire (pts (xy 180.34 102.87) (xy 191.77 102.87))
     (stroke (width 0) (type default))
   )
-  (wire (pts (xy 124.46 102.87) (xy 130.81 102.87))
-    (stroke (width 0) (type default))
-  )
-  (wire (pts (xy 130.81 91.44) (xy 130.81 87.63))
+  (wire (pts (xy 102.87 102.87) (xy 109.22 102.87))
+    (stroke (width 0) (type default))
+  )
+  (wire (pts (xy 109.22 91.44) (xy 109.22 87.63))
     (stroke (width 0) (type default))
   )
@@
     (stroke (width 0) (type default))
   )
-  (wire (pts (xy 124.46 92.71) (xy 121.92 92.71))
-    (stroke (width 0) (type default))
-  )
-  (wire (pts (xy 130.81 102.87) (xy 173.99 102.87))
-    (stroke (width 0) (type default))
-  )
-  (wire (pts (xy 130.81 87.63) (xy 138.43 87.63))
+  (wire (pts (xy 102.87 92.71) (xy 100.33 92.71))
+    (stroke (width 0) (type default))
+  )
+  (wire (pts (xy 109.22 87.63) (xy 115.57 87.63))
+    (stroke (width 0) (type default))
+  )
+  (wire (pts (xy 109.22 102.87) (xy 120.65 102.87))
     (stroke (width 0) (type default))
   )
@@
     (stroke (width 0) (type default))
   )
+  (wire (pts (xy 125.73 87.63) (xy 134.62 87.63))
+    (stroke (width 0) (type default))
+  )
   (wire (pts (xy 173.99 102.87) (xy 180.34 102.87))
     (stroke (width 0) (type default))
@@
     (stroke (width 0) (type default))
   )
-  (wire (pts (xy 124.46 90.17) (xy 121.92 90.17))
+  (wire (pts (xy 102.87 90.17) (xy 100.33 90.17))
     (stroke (width 0) (type default))
   )
@@
     (stroke (width 0) (type default))
   )
+  (wire (pts (xy 134.62 87.63) (xy 138.43 87.63))
+    (stroke (width 0) (type default))
+  )
+  (wire (pts (xy 120.65 102.87) (xy 173.99 102.87))
+    (stroke (width 0) (type default))
+  )
   (wire (pts (xy 191.77 87.63) (xy 191.77 80.01))
     (stroke (width 0) (type default))
   )
-  (wire (pts (xy 121.92 87.63) (xy 130.81 87.63))
-    (stroke (width 0) (type default))
-  )
-  (wire (pts (xy 124.46 92.71) (xy 124.46 102.87))
-    (stroke (width 0) (type default))
-  )
-  (wire (pts (xy 124.46 90.17) (xy 124.46 92.71))
-    (stroke (width 0) (type default))
-  )
-  (wire (pts (xy 130.81 99.06) (xy 130.81 102.87))
+  (wire (pts (xy 100.33 87.63) (xy 109.22 87.63))
+    (stroke (width 0) (type default))
+  )
+  (wire (pts (xy 102.87 92.71) (xy 102.87 102.87))
+    (stroke (width 0) (type default))
+  )
+  (wire (pts (xy 102.87 90.17) (xy 102.87 92.71))
+    (stroke (width 0) (type default))
+  )
+  (wire (pts (xy 120.65 95.25) (xy 120.65 102.87))
+    (stroke (width 0) (type default))
+  )
+  (wire (pts (xy 109.22 99.06) (xy 109.22 102.87))
     (stroke (width 0) (type default))
   )
@@
     )
   )
-  (netclass_flag "" (length 1) (shape dot) (at 134.62 87.63 0) (fields_autoplaced)
+  (netclass_flag "" (length 1) (shape dot) (at 109.22 87.63 0) (fields_autoplaced)
     (effects (font (size 1.27 1.27) (color 255 0 0 1)) (justify left bottom))
-    (property "Netclass" "Power" (at 135.3185 86.63 0)
-      (effects (font (size 1.27 1.27) italic) (justify left) hide)
-    )
-  )
-  (symbol (lib_id "jcap-symbols:PJ-202AH") (at 116.84 90.17 0) (unit 1)
+    (property "Netclass" "Power" (at 109.9185 86.63 0)
+      (effects (font (size 1.27 1.27) italic) (justify left) hide)
+    )
+  )
+  (netclass_flag "" (length 1) (shape dot) (at 134.62 87.63 180) (fields_autoplaced)
+    (effects (font (size 1.27 1.27) (color 255 0 0 1)) (justify right bottom))
+    (property "Netclass" "Power" (at 135.3185 88.63 0)
+      (effects (font (size 1.27 1.27) italic) (justify left) hide)
+    )
+  )
+  (symbol (lib_id "power:PWR_FLAG") (at 134.62 87.63 0) (unit 1)
     (in_bom yes) (on_board yes) (dnp no) (fields_autoplaced)
-    (property "Reference" "J301" (at 116.84 81.28 0)
-      (effects (font (size 1.27 1.27)))
-    )
-    (property "Value" "DC IN" (at 116.84 83.82 0)
-      (effects (font (size 1.27 1.27)))
-    )
-    (property "Footprint" "jcap-footprints:CUI_PJ-202AH" (at 116.84 90.17 0)
+    (property "Reference" "#FLG0301" (at 134.62 85.725 0)
+      (effects (font (size 1.27 1.27)) hide)
+    )
+    (property "Value" "PWR_FLAG" (at 134.62 82.55 0)
+      (effects (font (size 1.27 1.27)))
+    )
+    (property "Footprint" "" (at 134.62 87.63 0)
+      (effects (font (size 1.27 1.27)) hide)
+    )
+    (property "Datasheet" "~" (at 134.62 87.63 0)
+      (effects (font (size 1.27 1.27)) hide)
+    )
+    (pin "1")
+    (instances
+      (project "jcap"
+        (path "/7fc25e9e-3600-419b-89ef-b962e4e374c1/f5a50cf1-3d87-469f-beb1-b0b9cfae00ce"
+          (reference "#FLG0301") (unit 1)
+        )
+      )
+    )
+  )
+  (symbol (lib_id "jcap-symbols:PJ-202AH") (at 95.25 90.17 0) (unit 1)
+    (in_bom yes) (on_board yes) (dnp no) (fields_autoplaced)
+    (property "Reference" "J301" (at 95.25 81.28 0)
+      (effects (font (size 1.27 1.27)))
+    )
+    (property "Value" "DC IN" (at 95.25 83.82 0)
+      (effects (font (size 1.27 1.27)))
+    )
+    (property "Footprint" "jcap-footprints:CUI_PJ-202AH" (at 95.25 90.17 0)
       (effects (font (size 1.27 1.27)) (justify bottom) hide)
     )
-    (property "Datasheet" "~" (at 116.84 90.17 0)
-      (effects (font (size 1.27 1.27)) hide)
-    )
-    (pin "1")
-    (pin "2")
+    (property "Datasheet" "~" (at 95.25 90.17 0)
+      (effects (font (size 1.27 1.27)) hide)
+    )
     (pin "3")
+    (pin "1")
+    (pin "2")
     (instances
       (project "jcap"
@@
     )
   )
-  (symbol (lib_id "power:PWR_FLAG") (at 130.81 87.63 0) (unit 1)
+  (symbol (lib_id "Device:C") (at 109.22 95.25 180) (unit 1)
     (in_bom yes) (on_board yes) (dnp no) (fields_autoplaced)
-    (property "Reference" "#FLG0301" (at 130.81 85.725 0)
-      (effects (font (size 1.27 1.27)) hide)
-    )
-    (property "Value" "PWR_FLAG" (at 130.81 82.55 0)
-      (effects (font (size 1.27 1.27)))
-    )
-    (property "Footprint" "" (at 130.81 87.63 0)
-      (effects (font (size 1.27 1.27)) hide)
-    )
-    (property "Datasheet" "~" (at 130.81 87.63 0)
-      (effects (font (size 1.27 1.27)) hide)
-    )
-    (pin "1")
-    (instances
-      (project "jcap"
-        (path "/7fc25e9e-3600-419b-89ef-b962e4e374c1/f5a50cf1-3d87-469f-beb1-b0b9cfae00ce"
-          (reference "#FLG0301") (unit 1)
-        )
-      )
-    )
-  )
-  (symbol (lib_id "Device:C") (at 130.81 95.25 180) (unit 1)
-    (in_bom yes) (on_board yes) (dnp no) (fields_autoplaced)
-    (property "Reference" "C?" (at 134.62 93.98 0)
+    (property "Reference" "C?" (at 113.03 93.98 0)
       (effects (font (size 1.27 1.27)) (justify right))
     )
-    (property "Value" ".47u" (at 134.62 96.52 0)
+    (property "Value" ".47u" (at 113.03 96.52 0)
       (effects (font (size 1.27 1.27)) (justify right))
     )
-    (property "Footprint" "Capacitor_THT:C_Disc_D3.4mm_W2.1mm_P2.50mm" (at 129.8448 91.44 0)
-      (effects (font (size 1.27 1.27)) hide)
-    )
-    (property "Datasheet" "~" (at 130.81 95.25 0)
+    (property "Footprint" "Capacitor_THT:C_Disc_D3.4mm_W2.1mm_P2.50mm" (at 108.2548 91.44 0)
+      (effects (font (size 1.27 1.27)) hide)
+    )
+    (property "Datasheet" "~" (at 109.22 95.25 0)
       (effects (font (size 1.27 1.27)) hide)
     )
@@
     )
   )
-  (symbol (lib_id "power:PWR_FLAG") (at 130.81 102.87 180) (unit 1)
-    (in_bom yes) (on_board yes) (dnp no) (fields_autoplaced)
-    (property "Reference" "#FLG0302" (at 130.81 104.775 0)
-      (effects (font (size 1.27 1.27)) hide)
-    )
-    (property "Value" "PWR_FLAG" (at 130.81 107.95 0)
-      (effects (font (size 1.27 1.27)))
-    )
-    (property "Footprint" "" (at 130.81 102.87 0)
-      (effects (font (size 1.27 1.27)) hide)
-    )
-    (property "Datasheet" "~" (at 130.81 102.87 0)
-      (effects (font (size 1.27 1.27)) hide)
-    )
-    (pin "1")
-    (instances
-      (project "jcap"
-        (path "/7fc25e9e-3600-419b-89ef-b962e4e374c1/f5a50cf1-3d87-469f-beb1-b0b9cfae00ce"
-          (reference "#FLG0302") (unit 1)
-        )
-      )
+  (symbol (lib_id "jcap-symbols:IPP80P03P4L-04") (at 120.65 90.17 270) (mirror x) (unit 1)
+    (in_bom yes) (on_board yes) (dnp no)
+    (property "Reference" "Q301" (at 120.65 81.28 90)
+      (effects (font (size 1.27 1.27)))
+    )
+    (property "Value" "IPP80P03P4L-04" (at 120.65 83.82 90)
+      (effects (font (size 1.27 1.27)))
+    )
+    (property "Footprint" "Package_TO_SOT_THT:TO-220-3_Horizontal_TabDown" (at 118.745 83.82 0)
+      (effects (font (size 1.27 1.27) italic) (justify left) hide)
+    )
+    (property "Datasheet" "https://www.infineon.com/dgdl/Infineon-I80P03P4L_04-DataSheet-v01_01-EN.pdf?fileId=db3a30431ddc9372011e07e95eb827d7" (at 120.65 90.17 0)
+      (effects (font (size 1.27 1.27)) (justify left) hide)
+    )
+    (pin "1")
+    (pin "2")
+    (pin "3")
+    (instances
+      (project "jcap"
+        (path "/7fc25e9e-3600-419b-89ef-b962e4e374c1/f5a50cf1-3d87-469f-beb1-b0b9cfae00ce"
+          (reference "Q301") (unit 1)
+        )
+      )
